File: electronics/sensor-board/op_amp_array_6_lmc6036.kicad_sch (KiCad schematic)
At the start: 21 parts

Commit message: sensor-board edit
Parts:
- removed U? (x5): MAX44252ASD, symbol MAX44252ASD_Custom:MAX44252ASD
- added U? (x5): LMC6036, LMC6036:SOP65P640X120-14N, symbol LMC6036_custom:LMC6036
Connections:
- net VDD: now also U?.4 (VDD)
- net VSS: now also U?.11 (VSS)
- net output_A: now also U?.1 (OUTA)
- net output_B: now also U?.7 (OUTB)
- net output_C: now also U?.8 (OUTC)
- net output_D: now also U?.14 (OUTD)
- net at R?.1: now also U?.3 (INA+)
- net at R?.1, R?.2: now also U?.9 (INC-)
- net at R?.1: now also U?.10 (INC+)
- net at R?.1, R?.2: now also U?.13 (IND-)
- net at R?.1, R?.2: now also U?.2 (INA-)
- net at R?.1: now also U?.5 (INB+)
- net at R?.1, R?.2: now also U?.6 (INB-)
- net at R?.1: now also U?.12 (IND+)
Changed lines of the file:
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@@
   (junction (at 134.62 120.65) (diameter 0) (color 0 0 0 0))
   (junction (at 134.62 148.59) (diameter 0) (color 0 0 0 0))
-  (junction (at 147.32 60.96) (diameter 0) (color 0 0 0 0))
-  (junction (at 147.32 87.63) (diameter 0) (color 0 0 0 0))
-  (junction (at 147.32 115.57) (diameter 0) (color 0 0 0 0))
-  (junction (at 147.32 143.51) (diameter 0) (color 0 0 0 0))
-  (junction (at 162.56 63.5) (diameter 0) (color 0 0 0 0))
-  (junction (at 162.56 90.17) (diameter 0) (color 0 0 0 0))
-  (junction (at 162.56 118.11) (diameter 0) (color 0 0 0 0))
-  (junction (at 162.56 146.05) (diameter 0) (color 0 0 0 0))
   (wire (pts (xy 125.73 60.96) (xy 135.89 60.96))
     (stroke (width 0) (type default) (color 0 0 0 0))
@@
     (pin "2")
   )
-  (symbol (lib_id "MAX44252ASD_Custom:MAX44252ASD") (at 153.67 44.45 90) (unit 1)
+  (symbol (lib_id "LMC6036_custom:LMC6036") (at 153.67 44.45 90) (unit 5)
     (in_bom yes) (on_board yes) (fields_autoplaced)
     (property "Reference" "U?" (id 0) (at 153.67 35.56 90))
-    (property "Value" "MAX44252ASD" (id 1) (at 153.67 38.1 90))
-    (property "Footprint" "" (id 2) (at 153.67 42.545 0)
+    (property "Value" "LMC6036" (id 1) (at 153.67 38.1 90))
+    (property "Footprint" "LMC6036:SOP65P640X120-14N" (id 2) (at 153.67 42.545 0)
       (effects (font (size 1.27 1.27)) hide)
     )
@@
       (effects (font (size 1.27 1.27)) hide)
     )
+    (pin "11")
+    (pin "4")
+  )
+  (symbol (lib_id "LMC6036_custom:LMC6036") (at 153.67 63.5 0) (unit 1)
+    (in_bom yes) (on_board yes) (fields_autoplaced)
+    (property "Reference" "U?" (id 0) (at 154.94 53.34 0))
+    (property "Value" "LMC6036" (id 1) (at 154.94 55.88 0))
+    (property "Footprint" "LMC6036:SOP65P640X120-14N" (id 2) (at 155.575 63.5 0)
+      (effects (font (size 1.27 1.27)) hide)
+    )
+    (property "Datasheet" "" (id 3) (at 155.575 63.5 0)
+      (effects (font (size 1.27 1.27)) hide)
+    )
     (pin "1")
     (pin "2")
     (pin "3")
   )
-  (symbol (lib_id "MAX44252ASD_Custom:MAX44252ASD") (at 153.67 63.5 0) (unit 1)
-    (in_bom yes) (on_board yes)
-    (property "Reference" "U?" (id 0) (at 153.67 63.5 0))
-    (property "Value" "MAX44252ASD" (id 1) (at 154.94 55.88 0)
-      (effects (font (size 1.27 1.27)) hide)
-    )
-    (property "Footprint" "" (id 2) (at 155.575 63.5 0)
-      (effects (font (size 1.27 1.27)) hide)
-    )
-    (property "Datasheet" "" (id 3) (at 155.575 63.5 0)
-      (effects (font (size 1.27 1.27)) hide)
-    )
-    (pin "1")
-    (pin "2")
-    (pin "3")
-  )
-  (symbol (lib_id "MAX44252ASD_Custom:MAX44252ASD") (at 153.67 90.17 0) (unit 1)
-    (in_bom yes) (on_board yes)
-    (property "Reference" "U?" (id 0) (at 153.67 90.17 0))
-    (property "Value" "MAX44252ASD" (id 1) (at 154.94 82.55 0)
-      (effects (font (size 1.27 1.27)) hide)
-    )
-    (property "Footprint" "" (id 2) (at 155.575 90.17 0)
+  (symbol (lib_id "LMC6036_custom:LMC6036") (at 153.67 90.17 0) (unit 2)
+    (in_bom yes) (on_board yes) (fields_autoplaced)
+    (property "Reference" "U?" (id 0) (at 154.94 80.01 0))
+    (property "Value" "LMC6036" (id 1) (at 154.94 82.55 0))
+    (property "Footprint" "LMC6036:SOP65P640X120-14N" (id 2) (at 155.575 90.17 0)
       (effects (font (size 1.27 1.27)) hide)
     )
@@
       (effects (font (size 1.27 1.27)) hide)
     )
-    (pin "1")
-    (pin "2")
-    (pin "3")
-  )
-  (symbol (lib_id "MAX44252ASD_Custom:MAX44252ASD") (at 153.67 118.11 0) (unit 1)
-    (in_bom yes) (on_board yes)
-    (property "Reference" "U?" (id 0) (at 153.67 118.11 0))
-    (property "Value" "MAX44252ASD" (id 1) (at 154.94 110.49 0)
-      (effects (font (size 1.27 1.27)) hide)
-    )
-    (property "Footprint" "" (id 2) (at 155.575 118.11 0)
+    (pin "5")
+    (pin "6")
+    (pin "7")
+  )
+  (symbol (lib_id "LMC6036_custom:LMC6036") (at 153.67 118.11 0) (unit 3)
+    (in_bom yes) (on_board yes) (fields_autoplaced)
+    (property "Reference" "U?" (id 0) (at 154.94 107.95 0))
+    (property "Value" "LMC6036" (id 1) (at 154.94 110.49 0))
+    (property "Footprint" "LMC6036:SOP65P640X120-14N" (id 2) (at 155.575 118.11 0)
       (effects (font (size 1.27 1.27)) hide)
     )
@@
       (effects (font (size 1.27 1.27)) hide)
     )
-    (pin "1")
-    (pin "2")
-    (pin "3")
-  )
-  (symbol (lib_id "MAX44252ASD_Custom:MAX44252ASD") (at 153.67 146.05 0) (unit 1)
-    (in_bom yes) (on_board yes)
-    (property "Reference" "U?" (id 0) (at 153.67 146.05 0))
-    (property "Value" "MAX44252ASD" (id 1) (at 154.94 138.43 0)
-      (effects (font (size 1.27 1.27)) hide)
-    )
-    (property "Footprint" "" (id 2) (at 155.575 146.05 0)
+    (pin "10")
+    (pin "8")
+    (pin "9")
+  )
+  (symbol (lib_id "LMC6036_custom:LMC6036") (at 153.67 146.05 0) (unit 4)
+    (in_bom yes) (on_board yes) (fields_autoplaced)
+    (property "Reference" "U?" (id 0) (at 154.94 135.89 0))
+    (property "Value" "LMC6036" (id 1) (at 154.94 138.43 0))
+    (property "Footprint" "LMC6036:SOP65P640X120-14N" (id 2) (at 155.575 146.05 0)
       (effects (font (size 1.27 1.27)) hide)
     )
@@
       (effects (font (size 1.27 1.27)) hide)
     )
-    (pin "1")
-    (pin "2")
-    (pin "3")
-  )
-  (sheet_instances
-    (path "/" (page "1"))
-  )
-  (symbol_instances
-    (path "/16f7f778-8b07-4c2f-9dca-d8f867c210ec"
-      (reference "#PWR?") (unit 1) (value "GND") (footprint "")
-    )
-    (path "/373f77a2-94d8-40e6-8241-a306c1243b73"
-      (reference "#PWR?") (unit 1) (value "GND") (footprint "")
-    )
-    (path "/ae8e89ed-fa26-4694-a091-2db224c813b2"
-      (reference "#PWR?") (unit 1) (value "GND") (footprint "")
-    )
-    (path "/f2305714-43e0-4618-af93-91d034ff0c82"
-      (reference "#PWR?") (unit 1) (value "GND") (footprint "")
-    )
-    (path "/01e516df-4b4f-4517-bde7-da6fcdde2a4f"
-      (reference "R?") (unit 1) (value "R") (footprint "")
-    )
-    (path "/1688ae91-6e8e-4120-9669-4d0ca6d76832"
-      (reference "R?") (unit 1) (value "R") (footprint "")
-    )
-    (path "/63de2aad-f668-4325-9908-db4199b6d076"
-      (reference "R?") (unit 1) (value "R") (footprint "")
-    )
-    (path "/66f12ab2-0712-4942-8e16-8a0f1bf4c07b"
-      (reference "R?") (unit 1) (value "R") (footprint "")
-    )
-    (path "/6c159cba-3c9c-4abb-99bc-a123fce1e1fc"
-      (reference "R?") (unit 1) (value "R") (footprint "")
-    )
-    (path "/6ee274f2-bc66-4374-971a-a15bf2535e46"
-      (reference "R?") (unit 1) (value "R") (footprint "")
-    )
-    (path "/8215ebe9-31ed-4618-8a03-52406b30c840"
-      (reference "R?") (unit 1) (value "R") (footprint "")
-    )
-    (path "/89011c12-e113-4f61-a4f5-ba92ed02be93"
-      (reference "R?") (unit 1) (value "R") (footprint "")
-    )
-    (path "/93925990-b11c-4796-9637-ceb6f4ca45f3"
-      (reference "R?") (unit 1) (value "R") (footprint "")
-    )
-    (path "/a2754056-98eb-4794-9dc8-9ea71be49d01"
-      (reference "R?") (unit 1) (value "R") (footprint "")
-    )
-    (path "/a967f099-2ad0-429f-b4b9-adb50aee64e3"
-      (reference "R?") (unit 1) (value "R") (footprint "")
-    )
-    (path "/aa4ac85e-2e8c-4185-828f-9b0af10cb333"
-      (reference "R?") (unit 1) (value "R") (footprint "")
-    )
-    (path "/b2c90e11-4b04-4931-a917-ad8b76b05ddc"
-      (reference "R?") (unit 1) (value "R") (footprint "")
-    )
-    (path "/ca0c5e51-abd5-49b2-bedc-9b35d2d57dc2"
-      (reference "R?") (unit 1) (value "R") (footprint "")
-    )
-    (path "/ed8062f1-ffb4-442c-b553-c5ab7c35894f"
-      (reference "R?") (unit 1) (value "R") (footprint "")
-    )
-    (path "/ee41aa7f-a8c6-45c8-8346-95e08e7fb6d4"
-      (reference "R?") (unit 1) (value "R") (footprint "")
-    )
-    (path "/73caf16e-2004-4ed9-84a2-71b072b85c09"
-      (reference "U?") (unit 1) (value "MAX44252ASD") (footprint "")
-    )
-    (path "/f40e150d-45e1-4ddc-aa0a-853395417499"
-      (reference "U?") (unit 2) (value "MAX44252ASD") (footprint "")
-    )
-    (path "/5d6bd069-7adf-4a23-bb05-0d89023d387c"
-      (reference "U?") (unit 3) (value "MAX44252ASD") (footprint "")
-    )
-    (path "/d9fd8f7c-82e3-4164-b8fd-7e7aa20a1284"
-      (reference "U?") (unit 4) (value "MAX44252ASD") (footprint "")
-    )
-    (path "/f0e8b943-1ebe-4b77-b286-184ba7c9a665"
-      (reference "U?") (unit 5) (value "MAX44252ASD") (footprint "")
-    )
+    (pin "12")
+    (pin "13")
+    (pin "14")
   )
 )
