File: electronics/sensor-board/max44252_thermocouple_1.kicad_sch (KiCad schematic)
At the start: 21 parts

Commit message: sensor-board edits
Finalized pressure and flow sensor circuits.
Reorganized schematics
Parts:
- removed R? (x16): R, symbol Device:R
- removed U? (x5): MAX44252ASD, symbol MAX44252ASD_Custom:MAX44252ASD
- added R? (x16): R, symbol Device:R
- added U? (x5): MAX44252ASD, symbol MAX44252ASD_Custom:MAX44252ASD
Connections:
- net GND: now also R?.2, R?.2, R?.2, R?.2
- net VDD: now also U?.4 (VDD)
- net VSS: now also U?.11 (VSS)
- net diff+A: now also R?.1, R?.2
- net diff+B: now also R?.1, R?.2
- net diff+C: now also R?.1, R?.2
- net diff+D: now also R?.1, R?.2
- net diff-A: now also R?.2
- net diff-B: now also R?.2
- net diff-C: now also R?.2
- net diff-D: now also R?.2
- net output_A: now also R?.1, U?.1 (OUTA)
- net output_B: now also R?.1, U?.7 (OUTB)
- net output_C: now also R?.1, U?.8 (OUTC)
- net output_D: now also R?.1, U?.14 (OUTD)
- new net: R?.1, U?.10 (INC+)
- new net: R?.1, R?.2, U?.13 (IND-)
- new net: R?.1, U?.5 (INB+)
- new net: R?.1, R?.2, U?.6 (INB-)
- new net: R?.1, R?.2, U?.2 (INA-)
- new net: R?.1, U?.3 (INA+)
- new net: R?.1, R?.2, U?.9 (INC-)
- new net: R?.1, U?.12 (IND+)
Changed lines of the file:
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@@
     (pin "14")
   )
+  (sheet_instances
+    (path "/" (page "1"))
+  )
+  (symbol_instances
+    (path "/16f7f778-8b07-4c2f-9dca-d8f867c210ec"
+      (reference "#PWR?") (unit 1) (value "GND") (footprint "")
+    )
+    (path "/373f77a2-94d8-40e6-8241-a306c1243b73"
+      (reference "#PWR?") (unit 1) (value "GND") (footprint "")
+    )
+    (path "/ae8e89ed-fa26-4694-a091-2db224c813b2"
+      (reference "#PWR?") (unit 1) (value "GND") (footprint "")
+    )
+    (path "/f2305714-43e0-4618-af93-91d034ff0c82"
+      (reference "#PWR?") (unit 1) (value "GND") (footprint "")
+    )
+    (path "/01e516df-4b4f-4517-bde7-da6fcdde2a4f"
+      (reference "R?") (unit 1) (value "R") (footprint "")
+    )
+    (path "/1688ae91-6e8e-4120-9669-4d0ca6d76832"
+      (reference "R?") (unit 1) (value "R") (footprint "")
+    )
+    (path "/63de2aad-f668-4325-9908-db4199b6d076"
+      (reference "R?") (unit 1) (value "R") (footprint "")
+    )
+    (path "/66f12ab2-0712-4942-8e16-8a0f1bf4c07b"
+      (reference "R?") (unit 1) (value "R") (footprint "")
+    )
+    (path "/6c159cba-3c9c-4abb-99bc-a123fce1e1fc"
+      (reference "R?") (unit 1) (value "R") (footprint "")
+    )
+    (path "/6ee274f2-bc66-4374-971a-a15bf2535e46"
+      (reference "R?") (unit 1) (value "R") (footprint "")
+    )
+    (path "/8215ebe9-31ed-4618-8a03-52406b30c840"
+      (reference "R?") (unit 1) (value "R") (footprint "")
+    )
+    (path "/89011c12-e113-4f61-a4f5-ba92ed02be93"
+      (reference "R?") (unit 1) (value "R") (footprint "")
+    )
+    (path "/93925990-b11c-4796-9637-ceb6f4ca45f3"
+      (reference "R?") (unit 1) (value "R") (footprint "")
+    )
+    (path "/a2754056-98eb-4794-9dc8-9ea71be49d01"
+      (reference "R?") (unit 1) (value "R") (footprint "")
+    )
+    (path "/a967f099-2ad0-429f-b4b9-adb50aee64e3"
+      (reference "R?") (unit 1) (value "R") (footprint "")
+    )
+    (path "/aa4ac85e-2e8c-4185-828f-9b0af10cb333"
+      (reference "R?") (unit 1) (value "R") (footprint "")
+    )
+    (path "/b2c90e11-4b04-4931-a917-ad8b76b05ddc"
+      (reference "R?") (unit 1) (value "R") (footprint "")
+    )
+    (path "/ca0c5e51-abd5-49b2-bedc-9b35d2d57dc2"
+      (reference "R?") (unit 1) (value "R") (footprint "")
+    )
+    (path "/ed8062f1-ffb4-442c-b553-c5ab7c35894f"
+      (reference "R?") (unit 1) (value "R") (footprint "")
+    )
+    (path "/ee41aa7f-a8c6-45c8-8346-95e08e7fb6d4"
+      (reference "R?") (unit 1) (value "R") (footprint "")
+    )
+    (path "/73caf16e-2004-4ed9-84a2-71b072b85c09"
+      (reference "U?") (unit 1) (value "MAX44252ASD") (footprint "")
+    )
+    (path "/f40e150d-45e1-4ddc-aa0a-853395417499"
+      (reference "U?") (unit 2) (value "MAX44252ASD") (footprint "")
+    )
+    (path "/5d6bd069-7adf-4a23-bb05-0d89023d387c"
+      (reference "U?") (unit 3) (value "MAX44252ASD") (footprint "")
+    )
+    (path "/d9fd8f7c-82e3-4164-b8fd-7e7aa20a1284"
+      (reference "U?") (unit 4) (value "MAX44252ASD") (footprint "")
+    )
+    (path "/f0e8b943-1ebe-4b77-b286-184ba7c9a665"
+      (reference "U?") (unit 5) (value "MAX44252ASD") (footprint "")
+    )
+  )
 )
