File: electronics/sensor-board/sensor-board.kicad_pcb (KiCad board)
At the start: 4 copper layers, 168.7 x 121.2 mm, 189 parts, among them J1 SWD Header, J10 Suppply_5V, J11 Pressure_1, J12 Pressure_2, J13 Pressure_3, J14 Pressure_4, J15 Pressure_9, J16 Flow_1, J17 Flow_2, J18 CAN_Bus, J19 Spare_1, J2 Supply_24V, J20 Spare_2, J21 Spare_3, J22 Spare_4, J23 Therm_1, J24 Therm_4, J25 Therm_7, J26 Therm_2, J27 Therm_5, J28 Therm_3, J29 Therm_6, J3 Supply_12V, J30 Spare_HR_1, J31 Spare_HR_2, J4 Load_C_1, J5 Load_C_2, J6 Pressure_5, J7 Pressure_6, J8 Pressure_7, J9 Pressure_8, SW1 SW_Push_Dual, U1 LD3985M33R_SOT23, U10 MCP96RL01T, U11 LMC6036, U12 LMC6036, U13 LMC6036, U14 MAX44252ASD, U15 LMC6036, U2 21-0041-3-M_90-0096-8L_MXM, U3 STM32F105VBH6, U4 MCP96RL01T, U5 MCP96RL01T, U6 MCP96RL01T, U7 MCP96RL01T, U8 MCP96RL01T, U9 MCP96RL01T, Y1 Crystal_GND24

Commit message: work on sensor-board
Parts:
- U2: value 21-0041-3-M_90-0096-8L_MXM -> MAX33012EASA+
- moved J17 14.8 mm to (73.2, 132.0)
- moved R104 14.8 mm to (76.7, 135.8)
- moved C15 14.8 mm to (215.7, 62.6)
- moved C16 14.8 mm to (159.3, 62.6)
- moved C20 14.8 mm to (102.9, 62.6)
- moved C21 14.8 mm to (196.9, 62.6)
- moved C22 14.8 mm to (140.5, 62.6)
- moved C25 14.8 mm to (178.1, 62.6)
- moved C27 14.8 mm to (105.3, 81.3)
- moved C28 14.8 mm to (110.3, 111.1)
- moved C3 14.8 mm to (195.0, 85.7)
- moved J3 14.8 mm to (206.0, 94.1)
- moved J5 14.8 mm to (73.0, 96.0)
- moved R10 14.8 mm to (213.9, 69.1)
- moved R108 14.8 mm to (119.8, 78.5)
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Routing:
- net GND: track 297.5 -> 307.3 mm
- net /SPARE_gen_purp_amp/output_A: track 15.2 -> 14.1 mm
- net /SPARE_gen_purp_amp/output_D: track 15.1 -> 14.0 mm
- net /SPARE_gen_purp_amp/output_B: track 14.3 -> 13.4 mm
- net /SPARE_gen_purp_amp/output_C: track 14.2 -> 13.3 mm
- net +3V3: track 574.2 -> 573.5 mm
- net /ADC12_IN15: vias 3 -> 2
