File: electronics/sensor-board/max44252_loadcells.kicad_sch (KiCad schematic)
At the start: 17 parts, among them U15 MAX44252ASD

Commit message: work on sensor-board
Parts:
- removed U15: MAX44252ASD, MAX44252ASD-:MAX44252ASD&plus_, symbol MAX44252ASD_Custom:MAX44252ASD
- added U14: MAX44252ASD, MAX44252ASD-:MAX44252ASD&plus_, symbol MAX44252ASD_Custom:MAX44252ASD
Connections:
- net VDD: now also U14.4 (VDD)
- net VSS: now also U14.11 (VSS)
- net output_A: now also U14.1 (OUTA)
- net output_B: now also U14.7 (OUTB)
- net output_C: now also U14.8 (OUTC)
- net output_D: now also U14.14 (OUTD)
- net at R71.1, R75.1: now also U14.10 (INC+)
- net at R73.1, R77.1: now also U14.12 (IND+)
- net at R69.1, R76.1: now also U14.3 (INA+)
- net at R67.1, R74.1: now also U14.5 (INB+)
- net at R68.1, R78.2: now also U14.2 (INA-)
- net at R70.1, R80.2: now also U14.9 (INC-)
- net at R66.1, R79.2: now also U14.6 (INB-)
- net at R72.1, R81.2: now also U14.13 (IND-)
Changed lines of the file:
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@@
   (junction (at 146.05 115.57) (diameter 0) (color 0 0 0 0))
   (junction (at 146.05 120.65) (diameter 0) (color 0 0 0 0))
+  (junction (at 146.05 143.51) (diameter 0) (color 0 0 0 0))
   (junction (at 146.05 148.59) (diameter 0) (color 0 0 0 0))
-  (junction (at 147.32 143.51) (diameter 0) (color 0 0 0 0))
-  (junction (at 162.56 63.5) (diameter 0) (color 0 0 0 0))
   (junction (at 162.56 90.17) (diameter 0) (color 0 0 0 0))
-  (junction (at 162.56 118.11) (diameter 0) (color 0 0 0 0))
-  (junction (at 162.56 146.05) (diameter 0) (color 0 0 0 0))
   (wire (pts (xy 125.73 60.96) (xy 135.89 60.96))
     (stroke (width 0) (type default) (color 0 0 0 0))
@@
     (stroke (width 0) (type default) (color 0 0 0 0))
   )
-  (wire (pts (xy 143.51 143.51) (xy 147.32 143.51))
+  (wire (pts (xy 143.51 143.51) (xy 146.05 143.51))
     (stroke (width 0) (type default) (color 0 0 0 0))
   )
@@
     (stroke (width 0) (type default) (color 0 0 0 0))
   )
+  (wire (pts (xy 146.05 138.43) (xy 146.05 143.51))
+    (stroke (width 0) (type default) (color 0 0 0 0))
+  )
+  (wire (pts (xy 146.05 143.51) (xy 147.32 143.51))
+    (stroke (width 0) (type default) (color 0 0 0 0))
+  )
   (wire (pts (xy 146.05 148.59) (xy 146.05 149.86))
     (stroke (width 0) (type default) (color 0 0 0 0))
@@
     (stroke (width 0) (type default) (color 0 0 0 0))
   )
-  (wire (pts (xy 147.32 138.43) (xy 147.32 143.51))
-    (stroke (width 0) (type default) (color 0 0 0 0))
-  )
   (wire (pts (xy 149.86 55.88) (xy 146.05 55.88))
     (stroke (width 0) (type default) (color 0 0 0 0))
@@
     (stroke (width 0) (type default) (color 0 0 0 0))
   )
-  (wire (pts (xy 149.86 138.43) (xy 147.32 138.43))
+  (wire (pts (xy 149.86 138.43) (xy 146.05 138.43))
     (stroke (width 0) (type default) (color 0 0 0 0))
   )
@@
   )
   (wire (pts (xy 160.02 44.45) (xy 162.56 44.45))
+    (stroke (width 0) (type default) (color 0 0 0 0))
+  )
+  (wire (pts (xy 161.29 90.17) (xy 162.56 90.17))
     (stroke (width 0) (type default) (color 0 0 0 0))
   )
@@
   (symbol (lib_id "MAX44252ASD_Custom:MAX44252ASD") (at 153.67 44.45 90) (unit 5)
     (in_bom yes) (on_board yes) (fields_autoplaced)
-    (property "Reference" "U15" (id 0) (at 153.67 35.56 90))
+    (property "Reference" "U14" (id 0) (at 153.67 35.56 90))
     (property "Value" "MAX44252ASD" (id 1) (at 153.67 38.1 90))
     (property "Footprint" "MAX44252ASD-:MAX44252ASD&plus_" (id 2) (at 153.67 42.545 0)
@@
     (pin "4")
   )
-  (symbol (lib_id "MAX44252ASD_Custom:MAX44252ASD") (at 153.67 63.5 0) (unit 1)
-    (in_bom yes) (on_board yes)
-    (property "Reference" "U15" (id 0) (at 153.67 63.5 0))
-    (property "Value" "MAX44252ASD" (id 1) (at 154.94 55.88 0)
-      (effects (font (size 1.27 1.27)) hide)
-    )
-    (property "Footprint" "MAX44252ASD-:MAX44252ASD&plus_" (id 2) (at 155.575 63.5 0)
-      (effects (font (size 1.27 1.27)) hide)
-    )
-    (property "Datasheet" "" (id 3) (at 155.575 63.5 0)
-      (effects (font (size 1.27 1.27)) hide)
-    )
-    (pin "1")
-    (pin "2")
-    (pin "3")
-  )
-  (symbol (lib_id "MAX44252ASD_Custom:MAX44252ASD") (at 153.67 90.17 0) (unit 2)
-    (in_bom yes) (on_board yes)
-    (property "Reference" "U15" (id 0) (at 153.67 90.17 0))
-    (property "Value" "MAX44252ASD" (id 1) (at 154.94 82.55 0)
-      (effects (font (size 1.27 1.27)) hide)
-    )
-    (property "Footprint" "MAX44252ASD-:MAX44252ASD&plus_" (id 2) (at 155.575 90.17 0)
-      (effects (font (size 1.27 1.27)) hide)
-    )
-    (property "Datasheet" "" (id 3) (at 155.575 90.17 0)
+  (symbol (lib_id "MAX44252ASD_Custom:MAX44252ASD") (at 152.4 90.17 0) (unit 2)
+    (in_bom yes) (on_board yes)
+    (property "Reference" "U14" (id 0) (at 153.67 80.01 0))
+    (property "Value" "MAX44252ASD" (id 1) (at 152.4 86.36 0))
+    (property "Footprint" "MAX44252ASD-:MAX44252ASD&plus_" (id 2) (at 154.305 90.17 0)
+      (effects (font (size 1.27 1.27)) hide)
+    )
+    (property "Datasheet" "" (id 3) (at 154.305 90.17 0)
       (effects (font (size 1.27 1.27)) hide)
     )
@@
     (pin "7")
   )
+  (symbol (lib_id "MAX44252ASD_Custom:MAX44252ASD") (at 153.67 63.5 0) (unit 1)
+    (in_bom yes) (on_board yes)
+    (property "Reference" "U14" (id 0) (at 154.94 53.34 0))
+    (property "Value" "MAX44252ASD" (id 1) (at 154.94 58.42 0))
+    (property "Footprint" "MAX44252ASD-:MAX44252ASD&plus_" (id 2) (at 155.575 63.5 0)
+      (effects (font (size 1.27 1.27)) hide)
+    )
+    (property "Datasheet" "" (id 3) (at 155.575 63.5 0)
+      (effects (font (size 1.27 1.27)) hide)
+    )
+    (pin "1")
+    (pin "2")
+    (pin "3")
+  )
   (symbol (lib_id "MAX44252ASD_Custom:MAX44252ASD") (at 153.67 118.11 0) (unit 3)
     (in_bom yes) (on_board yes)
-    (property "Reference" "U15" (id 0) (at 153.67 118.11 0))
-    (property "Value" "MAX44252ASD" (id 1) (at 154.94 110.49 0)
-      (effects (font (size 1.27 1.27)) hide)
-    )
+    (property "Reference" "U14" (id 0) (at 154.94 107.95 0))
+    (property "Value" "MAX44252ASD" (id 1) (at 156.21 113.03 0))
     (property "Footprint" "MAX44252ASD-:MAX44252ASD&plus_" (id 2) (at 155.575 118.11 0)
       (effects (font (size 1.27 1.27)) hide)
@@
   (symbol (lib_id "MAX44252ASD_Custom:MAX44252ASD") (at 153.67 146.05 0) (unit 4)
     (in_bom yes) (on_board yes)
-    (property "Reference" "U15" (id 0) (at 153.67 146.05 0))
-    (property "Value" "MAX44252ASD" (id 1) (at 154.94 138.43 0)
-      (effects (font (size 1.27 1.27)) hide)
-    )
+    (property "Reference" "U14" (id 0) (at 154.94 135.89 0))
+    (property "Value" "MAX44252ASD" (id 1) (at 154.94 140.97 0))
     (property "Footprint" "MAX44252ASD-:MAX44252ASD&plus_" (id 2) (at 155.575 146.05 0)
       (effects (font (size 1.27 1.27)) hide)

Commit message: More work on sensor-board
Parts:
- R70, R72: value 100 -> NO_RES
- R71, R73: value 24.92 -> NO_RES
- R75, R77, R80, R81: value 82500 -> 0
Changed lines of the file:
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@@
   (symbol (lib_id "Device:R") (at 146.05 125.73 0) (unit 1)
     (in_bom yes) (on_board yes) (fields_autoplaced)
-    (property "Reference" "R75" (id 0) (at 148.59 124.4599 0)
-      (effects (font (size 1.27 1.27)) (justify left))
-    )
-    (property "Value" "82500" (id 1) (at 148.59 126.9999 0)
-      (effects (font (size 1.27 1.27)) (justify left))
+    (property "Reference" "R75" (id 0) (at 143.51 124.4599 0)
+      (effects (font (size 1.27 1.27)) (justify right))
+    )
+    (property "Value" "0" (id 1) (at 143.51 126.9999 0)
+      (effects (font (size 1.27 1.27)) (justify right))
     )
     (property "Footprint" "Resistor_SMD:R_0603_1608Metric" (id 2) (at 144.272 125.73 90)
@@
       (effects (font (size 1.27 1.27)) (justify left))
     )
-    (property "Value" "82500" (id 1) (at 148.59 154.9399 0)
+    (property "Value" "0" (id 1) (at 148.59 154.9399 0)
       (effects (font (size 1.27 1.27)) (justify left))
     )
@@
   )
   (symbol (lib_id "Device:R") (at 139.7 66.04 270) (unit 1)
-    (in_bom yes) (on_board yes)
-    (property "Reference" "R69" (id 0) (at 140.716 64.516 90))
-    (property "Value" "24.92" (id 1) (at 135.382 68.58 90))
+    (in_bom yes) (on_board yes) (fields_autoplaced)
+    (property "Reference" "R69" (id 0) (at 139.7 69.85 90))
+    (property "Value" "24.92" (id 1) (at 139.7 72.39 90))
     (property "Footprint" "Resistor_SMD:R_0603_1608Metric" (id 2) (at 139.7 64.262 90)
       (effects (font (size 1.27 1.27)) hide)
@@
   )
   (symbol (lib_id "Device:R") (at 139.7 148.59 270) (unit 1)
-    (in_bom yes) (on_board yes)
-    (property "Reference" "R73" (id 0) (at 140.716 147.066 90))
-    (property "Value" "24.92" (id 1) (at 135.382 151.13 90))
+    (in_bom yes) (on_board yes) (fields_autoplaced)
+    (property "Reference" "R73" (id 0) (at 139.7 152.4 90))
+    (property "Value" "NO_RES" (id 1) (at 139.7 154.94 90))
     (property "Footprint" "Resistor_SMD:R_0603_1608Metric" (id 2) (at 139.7 146.812 90)
       (effects (font (size 1.27 1.27)) hide)
@@
   )
   (symbol (lib_id "Device:R") (at 139.7 92.71 270) (unit 1)
-    (in_bom yes) (on_board yes)
-    (property "Reference" "R67" (id 0) (at 140.716 91.186 90))
-    (property "Value" "24.92" (id 1) (at 135.382 95.25 90))
+    (in_bom yes) (on_board yes) (fields_autoplaced)
+    (property "Reference" "R67" (id 0) (at 139.7 96.52 90))
+    (property "Value" "24.92" (id 1) (at 139.7 99.06 90))
     (property "Footprint" "Resistor_SMD:R_0603_1608Metric" (id 2) (at 139.7 90.932 90)
       (effects (font (size 1.27 1.27)) hide)
@@
       (effects (font (size 1.27 1.27)) (justify left))
     )
-    (property "Value" "82500" (id 1) (at 148.59 99.06 0)
+    (property "Value" "82500" (id 1) (at 148.59 99.0599 0)
       (effects (font (size 1.27 1.27)) (justify left))
     )
@@
     (in_bom yes) (on_board yes) (fields_autoplaced)
     (property "Reference" "R70" (id 0) (at 139.7 109.22 90))
-    (property "Value" "100" (id 1) (at 139.7 111.76 90))
+    (property "Value" "NO_RES" (id 1) (at 139.7 111.76 90))
     (property "Footprint" "Resistor_SMD:R_0603_1608Metric" (id 2) (at 139.7 113.792 90)
       (effects (font (size 1.27 1.27)) hide)
@@
   (symbol (lib_id "MAX44252ASD_Custom:MAX44252ASD") (at 153.67 63.5 0) (unit 1)
     (in_bom yes) (on_board yes)
-    (property "Reference" "U14" (id 0) (at 154.94 53.34 0))
-    (property "Value" "MAX44252ASD" (id 1) (at 154.94 58.42 0))
+    (property "Reference" "U14" (id 0) (at 153.67 63.5 0))
+    (property "Value" "MAX44252ASD" (id 1) (at 163.83 67.31 0))
     (property "Footprint" "MAX44252ASD-:MAX44252ASD&plus_" (id 2) (at 155.575 63.5 0)
       (effects (font (size 1.27 1.27)) hide)
@@
   (symbol (lib_id "MAX44252ASD_Custom:MAX44252ASD") (at 153.67 118.11 0) (unit 3)
     (in_bom yes) (on_board yes)
-    (property "Reference" "U14" (id 0) (at 154.94 107.95 0))
-    (property "Value" "MAX44252ASD" (id 1) (at 156.21 113.03 0))
+    (property "Reference" "U14" (id 0) (at 153.67 118.11 0))
+    (property "Value" "MAX44252ASD" (id 1) (at 162.56 121.92 0))
     (property "Footprint" "MAX44252ASD-:MAX44252ASD&plus_" (id 2) (at 155.575 118.11 0)
       (effects (font (size 1.27 1.27)) hide)
@@
   (symbol (lib_id "MAX44252ASD_Custom:MAX44252ASD") (at 153.67 146.05 0) (unit 4)
     (in_bom yes) (on_board yes)
-    (property "Reference" "U14" (id 0) (at 154.94 135.89 0))
-    (property "Value" "MAX44252ASD" (id 1) (at 154.94 140.97 0))
+    (property "Reference" "U14" (id 0) (at 153.67 146.05 0))
+    (property "Value" "MAX44252ASD" (id 1) (at 163.83 149.86 0))
     (property "Footprint" "MAX44252ASD-:MAX44252ASD&plus_" (id 2) (at 155.575 146.05 0)
       (effects (font (size 1.27 1.27)) hide)
@@
   (symbol (lib_id "MAX44252ASD_Custom:MAX44252ASD") (at 152.4 90.17 0) (unit 2)
     (in_bom yes) (on_board yes)
-    (property "Reference" "U14" (id 0) (at 153.67 80.01 0))
-    (property "Value" "MAX44252ASD" (id 1) (at 152.4 86.36 0))
+    (property "Reference" "U14" (id 0) (at 152.4 90.17 0))
+    (property "Value" "MAX44252ASD" (id 1) (at 162.56 93.98 0))
     (property "Footprint" "MAX44252ASD-:MAX44252ASD&plus_" (id 2) (at 154.305 90.17 0)
       (effects (font (size 1.27 1.27)) hide)
@@
     (in_bom yes) (on_board yes) (fields_autoplaced)
     (property "Reference" "R80" (id 0) (at 153.67 104.14 90))
-    (property "Value" "82500" (id 1) (at 153.67 106.68 90))
+    (property "Value" "0" (id 1) (at 153.67 106.68 90))
     (property "Footprint" "Resistor_SMD:R_0603_1608Metric" (id 2) (at 153.67 108.712 90)
       (effects (font (size 1.27 1.27)) hide)
@@
     (in_bom yes) (on_board yes) (fields_autoplaced)
     (property "Reference" "R72" (id 0) (at 139.7 137.16 90))
-    (property "Value" "100" (id 1) (at 139.7 139.7 90))
+    (property "Value" "NO_RES" (id 1) (at 139.7 139.7 90))
     (property "Footprint" "Resistor_SMD:R_0603_1608Metric" (id 2) (at 139.7 141.732 90)
       (effects (font (size 1.27 1.27)) hide)
@@
   )
   (symbol (lib_id "Device:R") (at 139.7 120.65 270) (unit 1)
-    (in_bom yes) (on_board yes)
-    (property "Reference" "R71" (id 0) (at 140.716 119.126 90))
-    (property "Value" "24.92" (id 1) (at 135.382 123.19 90))
+    (in_bom yes) (on_board yes) (fields_autoplaced)
+    (property "Reference" "R71" (id 0) (at 139.7 114.3 90))
+    (property "Value" "NO_RES" (id 1) (at 139.7 116.84 90))
     (property "Footprint" "Resistor_SMD:R_0603_1608Metric" (id 2) (at 139.7 118.872 90)
       (effects (font (size 1.27 1.27)) hide)
@@
     (in_bom yes) (on_board yes) (fields_autoplaced)
     (property "Reference" "R81" (id 0) (at 153.67 132.08 90))
-    (property "Value" "82500" (id 1) (at 153.67 134.62 90))
+    (property "Value" "0" (id 1) (at 153.67 134.62 90))
     (property "Footprint" "Resistor_SMD:R_0603_1608Metric" (id 2) (at 153.67 136.652 90)
       (effects (font (size 1.27 1.27)) hide)
