File: electronics/sensor-board/OLD DESIGN sensor-board.kicad_sch (KiCad schematic)
At the start: 83 parts, among them J1 Spare_HR_1, J10 Pressure_8, J11 Load_C_1, J12 Load_C_2, J13 Pressure_1, J14 Pressure_2, J15 Pressure_3, J16 Pressure_4, J17 Pressure_9, J18 Flow_1, J19 Flow_2, J2 Spare_HR_2, J20 Spare_1, J21 Spare_2, J22 Spare_3, J23 Spare_4, J24 CAN_Bus, J25 CAN_Bus, J3 SWD Header, J4 Suppply_5V, J5 Supply_24V, J6 Supply_12V, J7 Pressure_5, J8 Pressure_6, J9 Pressure_7, SW1 SW_Push_Dual, U1 LD3985M33R_SOT23, U2 STM32F105VBH6, U3 MAX33014EATB+, Y1 36 MHz

Commit message: updated loadcell amplifier
Parts:
- removed C3, C4: 100nF, Capacitor_SMD:C_0603_1608Metric, symbol Device:C_Small
- removed CR1, CR2, CR3: MM3Z3V6C, 3.3V Zener:MM3Z3V6C, symbol 3.3V Zener:MM3Z3V6C
- removed R1: 2.3k, Resistor_SMD:R_0603_1608Metric, symbol Device:R
- removed R2: 1k, Resistor_SMD:R_0603_1608Metric, symbol Device:R
- removed R3, R4: 200, Resistor_SMD:R_0603_1608Metric, symbol Device:R
- added U16: CZRF52C3V3, 3.3V Zener:CZRF52C3V3, symbol 3.3V Zener:CZRF52C3V3
- renumbered C13 to C10, C14 to C11, C6 to C12, C7 to C27, C8 to C28, C15 to C29, C5 to C3, C9 to C6, C10 to C7, C11 to C8, C12 to C9, D4 to D1, D1 to D2, D2 to D3, D3 to D4, J3 to J1, J4 to J10, J13 to J11, J14 to J12, J15 to J13, J16 to J14, J17 to J15, J18 to J16, J19 to J17, J24 to J18, J20 to J19, J5 to J2, J21 to J20, J22 to J21, J23 to J22, J6 to J3, J1 to J30, J2 to J31, J25 to J32, J11 to J4, J12 to J5, J7 to J6, J8 to J7, J9 to J8, J10 to J9, R13 to R1, R14 to R101, R15 to R105, R11 to R106, R12 to R107, R8 to R108, R9 to R109, R10 to R110, R5 to R111, R6 to R112, R7 to R2, TP2 to TP1, TP9 to TP10, TP1 to TP11, TP11 to TP12, TP12 to TP13, TP13 to TP14, TP14 to TP15, TP10 to TP16, TP3 to TP2, TP4 to TP3, TP5 to TP4, TP15 to TP5, TP6 to TP7, TP7 to TP8, TP8 to TP9, U3 to U2, U2 to U3
Connections:
- net ADC12_IN15: now also U16.1
- net GND: now also U16.2
- net Load Cell/output_D: now reaches TP11.1
- net Load Cell/diff+D: now reaches J31.2 (Pin_2)
- net Load Cell/diff-D: now reaches J31.3 (Pin_3)
- net Load Cell/diff+C: now reaches J30.2 (Pin_2)
- net Load Cell/diff-C: now reaches J30.3 (Pin_3)
- net Load Cell/In+ renamed Load Cell/diff-A
- net Load Cell/In- renamed Load Cell/diff+A
- net Load Cell 2/In+ renamed Load Cell/diff-B
- net Load Cell 2/In- renamed Load Cell/diff+B
Other:
- sheet Load Cell 1 renamed Load Cell
- removed sheet Load Cell 2
- sheet Load Cell: file max44252_loadcell1.kicad_sch -> max44252_loadcells.kicad_sch
- sheet Load Cell ports: added diff+A, diff+B, diff+C, diff+D, diff-A, diff-B, diff-C, diff-D, output_A, output_B, output_C, output_D; removed In+, In-, Vref, out
- moved on the sheet: J11, J12, J13, J14, J15, J16, J17, J19, J20, J21, J22, J30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
