File: electronics/output-board/output-board.kicad_sch (KiCad schematic)
At the start: 37 parts, among them J14 Arming switch, J3 12V In, J4 Conn_01x02, J5 SWD Header, J6 Conn_01x02, SW1 SW_Push_Dual, U1 MAX33012EASA+, U2 LD3985M33R_SOT23, U3 STM32F446ZEHx, Y1 25MHz 9pF

Commit message: Output Board is basically done!
Other:
- note added: "To Do: -Layout Board -Get Footprints"
- note removed: "To Do: -Servo Valve Control? -Layout Board -Get Footprints"
Changed lines of the file:
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@@
 (kicad_sch (version 20210621) (generator eeschema)
   (paper "A2")
-  (junction (at 25.4 140.97) (diameter 0) (color 0 0 0 0))
   (junction (at 25.4 152.4) (diameter 0) (color 0 0 0 0))
   (junction (at 25.4 163.83) (diameter 0) (color 0 0 0 0))
@@
   (junction (at 25.4 220.98) (diameter 0) (color 0 0 0 0))
   (junction (at 25.4 232.41) (diameter 0) (color 0 0 0 0))
+  (junction (at 25.4 243.84) (diameter 0) (color 0 0 0 0))
   (junction (at 26.67 278.13) (diameter 0) (color 0 0 0 0))
   (junction (at 26.67 289.56) (diameter 0) (color 0 0 0 0))
@@
     (stroke (width 0) (type solid) (color 0 0 0 0))
   )
-  (wire (pts (xy 25.4 137.16) (xy 25.4 140.97))
-    (stroke (width 0) (type default) (color 0 0 0 0))
-  )
   (wire (pts (xy 25.4 140.97) (xy 25.4 152.4))
     (stroke (width 0) (type default) (color 0 0 0 0))
@@
   )
   (wire (pts (xy 25.4 243.84) (xy 25.4 232.41))
+    (stroke (width 0) (type default) (color 0 0 0 0))
+  )
+  (wire (pts (xy 25.4 243.84) (xy 25.4 250.19))
     (stroke (width 0) (type default) (color 0 0 0 0))
   )
@@
     (effects (font (size 1.27 1.27)) (justify left bottom))
   )
-  (text "To Do:\n\n-Servo Valve Control?\n-Layout Board\n-Get Footprints"
-    (at 295.91 144.78 0)
+  (text "To Do:\n\n-Layout Board\n-Get Footprints" (at 295.91 144.78 0)
     (effects (font (size 10 10)) (justify left bottom))
   )
@@
     (pin "1")
   )
-  (symbol (lib_id "power:+12V") (at 25.4 137.16 0) (unit 1)
-    (in_bom yes) (on_board yes) (fields_autoplaced)
-    (property "Reference" "#PWR0107" (id 0) (at 25.4 140.97 0)
-      (effects (font (size 1.27 1.27)) hide)
-    )
-    (property "Value" "+12V" (id 1) (at 25.4 133.5554 0))
-    (property "Footprint" "" (id 2) (at 25.4 137.16 0)
-      (effects (font (size 1.27 1.27)) hide)
-    )
-    (property "Datasheet" "" (id 3) (at 25.4 137.16 0)
-      (effects (font (size 1.27 1.27)) hide)
-    )
-    (pin "1")
-  )
   (symbol (lib_id "power:+12V") (at 30.48 326.39 180) (unit 1)
     (in_bom yes) (on_board yes)
@@
     )
     (property "Datasheet" "" (id 3) (at 228.6 52.07 0)
+      (effects (font (size 1.27 1.27)) hide)
+    )
+    (pin "1")
+  )
+  (symbol (lib_id "power:GND") (at 25.4 250.19 0) (unit 1)
+    (in_bom yes) (on_board yes) (fields_autoplaced)
+    (property "Reference" "#PWR0107" (id 0) (at 25.4 256.54 0)
+      (effects (font (size 1.27 1.27)) hide)
+    )
+    (property "Value" "GND" (id 1) (at 25.4 254.7526 0))
+    (property "Footprint" "" (id 2) (at 25.4 250.19 0)
+      (effects (font (size 1.27 1.27)) hide)
+    )
+    (property "Datasheet" "" (id 3) (at 25.4 250.19 0)
       (effects (font (size 1.27 1.27)) hide)
     )
@@
       (reference "#PWR0106") (unit 1) (value "GND") (footprint "")
     )
-    (path "/f690d10e-42b3-4dcd-b346-4624f5ab1baa"
-      (reference "#PWR0107") (unit 1) (value "+12V") (footprint "")
+    (path "/7eac883b-36e6-4fe4-9374-3a11d80f879d"
+      (reference "#PWR0107") (unit 1) (value "GND") (footprint "")
     )
     (path "/bd87855a-783c-4e33-a6c0-125ff9084867"
@@
     )
     (path "/36b6bf08-79b4-4cbd-9663-410f8ea161a3/6b60855c-5bd9-463e-a130-45a0cde73160"
-      (reference "J1") (unit 1) (value "Conn_01x02_Male") (footprint "Connector_Molex:Molex_SL_171971-0002_1x02_P2.54mm_Vertical")
+      (reference "J1") (unit 1) (value "Conn_01x02_Male") (footprint "Connector_PinHeader_2.54mm:PinHeader_1x02_P2.54mm_Horizontal")
     )
     (path "/7c0b44ed-3289-4df7-a2ca-32e0eb184fe3/6b60855c-5bd9-463e-a130-45a0cde73160"
-      (reference "J2") (unit 1) (value "Conn_01x02_Male") (footprint "Connector_Molex:Molex_SL_171971-0002_1x02_P2.54mm_Vertical")
+      (reference "J2") (unit 1) (value "Conn_01x02_Male") (footprint "Connector_PinHeader_2.54mm:PinHeader_1x02_P2.54mm_Horizontal")
     )
     (path "/4598fa52-b178-42fa-b08e-f370d8204e39"
@@
     )
     (path "/1ea806a6-f443-4e80-87ef-b585f08de103/6b60855c-5bd9-463e-a130-45a0cde73160"
-      (reference "J7") (unit 1) (value "Conn_01x02_Male") (footprint "Connector_Molex:Molex_SL_171971-0002_1x02_P2.54mm_Vertical")
+      (reference "J7") (unit 1) (value "Conn_01x02_Male") (footprint "Connector_PinHeader_2.54mm:PinHeader_1x02_P2.54mm_Horizontal")
     )
     (path "/95861652-6caa-440d-ae33-35c3e6668a9b/6b60855c-5bd9-463e-a130-45a0cde73160"
-      (reference "J8") (unit 1) (value "Conn_01x02_Male") (footprint "Connector_Molex:Molex_SL_171971-0002_1x02_P2.54mm_Vertical")
+      (reference "J8") (unit 1) (value "Conn_01x02_Male") (footprint "Connector_PinHeader_2.54mm:PinHeader_1x02_P2.54mm_Horizontal")
     )
     (path "/59ac11d2-41f8-4525-b5e6-c9b69cc3d64d/6b60855c-5bd9-463e-a130-45a0cde73160"
-      (reference "J9") (unit 1) (value "Conn_01x02_Male") (footprint "Connector_Molex:Molex_SL_171971-0002_1x02_P2.54mm_Vertical")
+      (reference "J9") (unit 1) (value "Conn_01x02_Male") (footprint "Connector_PinHeader_2.54mm:PinHeader_1x02_P2.54mm_Horizontal")
     )
     (path "/fa9df34d-6cdc-4ba2-a240-df8a947a170c/6b60855c-5bd9-463e-a130-45a0cde73160"
-      (reference "J10") (unit 1) (value "Conn_01x02_Male") (footprint "Connector_Molex:Molex_SL_171971-0002_1x02_P2.54mm_Vertical")
+      (reference "J10") (unit 1) (value "Conn_01x02_Male") (footprint "Connector_PinHeader_2.54mm:PinHeader_1x02_P2.54mm_Horizontal")
     )
     (path "/fd555d38-9efd-4090-b580-398f0ce3794c/6b60855c-5bd9-463e-a130-45a0cde73160"
-      (reference "J11") (unit 1) (value "Conn_01x02_Male") (footprint "Connector_Molex:Molex_SL_171971-0002_1x02_P2.54mm_Vertical")
+      (reference "J11") (unit 1) (value "Conn_01x02_Male") (footprint "Connector_PinHeader_2.54mm:PinHeader_1x02_P2.54mm_Horizontal")
     )
     (path "/b1c0de20-a4c8-4523-b668-2cf58a13b8ef/6b60855c-5bd9-463e-a130-45a0cde73160"
-      (reference "J12") (unit 1) (value "Conn_01x02_Male") (footprint "Connector_Molex:Molex_SL_171971-0002_1x02_P2.54mm_Vertical")
+      (reference "J12") (unit 1) (value "Conn_01x02_Male") (footprint "Connector_PinHeader_2.54mm:PinHeader_1x02_P2.54mm_Horizontal")
     )
     (path "/ca1ddf89-c899-4fe9-b54d-3dccafa5d0cc/6b60855c-5bd9-463e-a130-45a0cde73160"
-      (reference "J13") (unit 1) (value "Conn_01x02_Male") (footprint "Connector_Molex:Molex_SL_171971-0002_1x02_P2.54mm_Vertical")
+      (reference "J13") (unit 1) (value "Conn_01x02_Male") (footprint "Connector_PinHeader_2.54mm:PinHeader_1x02_P2.54mm_Horizontal")
     )
     (path "/dae9d700-6159-4d31-9d5b-15df687ec690"
@@
     )
     (path "/f63df9f3-f635-4488-812a-e53c82698e77/6b60855c-5bd9-463e-a130-45a0cde73160"
-      (reference "J15") (unit 1) (value "Conn_01x02_Male") (footprint "Connector_Molex:Molex_SL_171971-0002_1x02_P2.54mm_Vertical")
+      (reference "J15") (unit 1) (value "Conn_01x02_Male") (footprint "Connector_PinHeader_2.54mm:PinHeader_1x02_P2.54mm_Horizontal")
     )
     (path "/1b6584c1-0d12-464b-be81-0b19bbe2e291/6b60855c-5bd9-463e-a130-45a0cde73160"
-      (reference "J16") (unit 1) (value "Conn_01x02_Male") (footprint "Connector_Molex:Molex_SL_171971-0002_1x02_P2.54mm_Vertical")
+      (reference "J16") (unit 1) (value "Conn_01x02_Male") (footprint "Connector_PinHeader_2.54mm:PinHeader_1x02_P2.54mm_Horizontal")
     )
     (path "/03ffcab8-edae-43b1-a3a4-8f66704c20eb/6b60855c-5bd9-463e-a130-45a0cde73160"
-      (reference "J17") (unit 1) (value "Conn_01x02_Male") (footprint "Connector_Molex:Molex_SL_171971-0002_1x02_P2.54mm_Vertical")
+      (reference "J17") (unit 1) (value "Conn_01x02_Male") (footprint "Connector_PinHeader_2.54mm:PinHeader_1x02_P2.54mm_Horizontal")
     )
     (path "/691537aa-0e14-4c5f-8530-ba42c3dce2d9/6b60855c-5bd9-463e-a130-45a0cde73160"
-      (reference "J18") (unit 1) (value "Conn_01x02_Male") (footprint "Connector_Molex:Molex_SL_171971-0002_1x02_P2.54mm_Vertical")
+      (reference "J18") (unit 1) (value "Conn_01x02_Male") (footprint "Connector_PinHeader_2.54mm:PinHeader_1x02_P2.54mm_Horizontal")
     )
     (path "/b06f02ce-a9d0-4544-ada1-f271ca89a2cc"

Commit message: Put in connectors and finalized layout of everything except MCU.
Parts:
- added J19: Extra IO, Connector_PinHeader_2.54mm:PinHeader_2x03_P2.54mm_Vertical, symbol Connector:Conn_01x06_Male
- J14, J4, J6: footprint Connector_PinHeader_2.54mm:PinHeader_1x02_P2.54mm_Vertical -> CustomFootprints:LatchingConnector2POS
- J3: footprint Connector_PinHeader_2.54mm:PinHeader_1x02_P2.54mm_Vertical -> CustomFootprints:PowerPoleThroughHole
Connections:
- net +5V: now also J4.2 (Pin_2); no longer J4.1 (Pin_1)
- net GND: now also J4.1 (Pin_1); no longer J4.2 (Pin_2)
Other:
- note added: "To Do: -Find MCU -Add IO Breakout -Finalize Connectors -Put together final parrts list -Buy parts and board"
- note removed: "To Do: -Layout Board -Get Footprints"

Commit message: Updated MCU Base and started MCU on Output Board
Parts:
- removed C14, C15, C16, C17, C18, C19, C20, C21: 100nF, Capacitor_SMD:C_0603_1608Metric, symbol Device:C_Small
- removed U3: STM32F446ZEHx, Package_BGA:UFBGA-144_7x7mm_Layout12x12_P0.5mm, symbol MCU_ST_STM32F4:STM32F446ZEHx
- added U3: STM32F105VBH6, Package_BGA:LFBGA-100_10x10mm_Layout10x10_P0.8mm, symbol F105 MCU:STM32F105VBH6
- C10, C11: value 100nF -> 20pF
- C4, C5: value 20pF -> 100nF
- C7, C8: value 2.2uF -> 100nF
- R1: value 0k -> 10k
- R3: value 10k -> 0k
Connections:
- net +3V3: now also C4.1, C5.1, C8.1, U3.B2 (VBAT), U3.D2 (VDD_5), U3.F4 (VDD_4), U3.F5 (VDD_3), U3.F6 (VDD_2), U3.F7 (VDD_1); no longer C11.1
- net CAN_RX: now also U3.C10 (PA11)
- net CAN_TX: now also U3.B10 (PA12)
- net GND: now also C10.1, C11.1, C4.2, C5.2, C6.2, R1.2, SW1.2, SW1.4, U3.C2 (VSS_5), U3.E4 (VSS_4), U3.E5 (VSS_3), U3.E6 (VSS_2), U3.E7 (VSS_1), U3.G1 (VSSA), U3.H1 (VREF-); no longer C10.2, C11.2, C4.1, C5.1, C6.1, R3.2, SW1.1, SW1.3
- net Ignition MOSFET/INPUT: now also U3.K8 (PB12)
- net MOSFET-sheet/INPUT: now also U3.J4 (PB0)
- net MOSFET-sheet1/INPUT: now also U3.K4 (PB1)
- net MOSFET-sheet10/INPUT: now also U3.J7 (PB10)
- net MOSFET-sheet11/INPUT: now also U3.K7 (PB11)
- net MOSFET-sheet2/INPUT: now also U3.G5 (PB2)
- net MOSFET-sheet3/INPUT: now also U3.A7 (PB3)
- net MOSFET-sheet4/INPUT: now also U3.A6 (PB4)
- net MOSFET-sheet5/INPUT: now also U3.C5 (PB5)
- net MOSFET-sheet6/INPUT: now also U3.B5 (PB6)
- net MOSFET-sheet7/INPUT: now also U3.A5 (PB7)
- net MOSFET-sheet8/INPUT: now also U3.B4 (PB8)
- net MOSFET-sheet9/INPUT: now also U3.A4 (PB9)
- net SWCLK: now also U3.A9 (PA14)
- net SWDIO: now also U3.A10 (PA13)
- net VDDA: now also C6.1, U3.J1 (VREF+), U3.K1 (VDDA); no longer C10.1
- net at J14.1 (Pin_1), R12.2: now also U3.G8 (PB15)
- net at Y1.1: now also C10.2, U3.C1 (OSC_IN); no longer C5.2
- net at R3.1: now also C11.2, Y1.2
- net at C7.1: now also SW1.1, SW1.3, U3.E1 (NRST)
- new net: R3.2, U3.D1 (OSC_OUT)
- new net: R1.1, U3.D5 (BOOT0)
Other:
- note removed: "Should be ceramic capacitors (low ESR)"
