File: electronics/datasheets/sensor-board/sensor-board.kicad_pcb (KiCad board)
At the start: 4 copper layers, 176.6 x 134.6 mm, 189 parts, among them J1 SWD Header, J10 Suppply_5V, J11 Pressure_1, J12 Pressure_2, J13 Pressure_3, J14 Pressure_4, J15 Pressure_9, J16 Flow_1, J17 Flow_2, J18 CAN_Bus, J19 Spare_1, J2 Supply_24V, J20 Spare_2, J21 Spare_3, J22 Spare_4, J23 Therm_1, J24 Therm_4, J25 Therm_7, J26 Therm_2, J27 Therm_5, J28 Therm_3, J29 Therm_6, J3 Supply_12V, J30 Spare_HR_1, J31 Spare_HR_2, J4 Load_C_1, J5 Load_C_2, J6 Pressure_5, J7 Pressure_6, J8 Pressure_7, J9 Pressure_8, SW1 SW_Push_Dual, U1 LD3985M33R_SOT23, U10 MCP96RL01T, U11 LMC6036, U12 LMC6036, U13 LMC6036, U14 MAX44252ASD, U15 LMC6036, U2 MAX33012EASA+, U3 STM32F105VBH6, U4 MCP96RL01T, U5 MCP96RL01T, U6 MCP96RL01T, U7 MCP96RL01T, U8 MCP96RL01T, U9 MCP96RL01T, Y1 Crystal_GND24

Commit message: Work on sensor-board
Parts:
- added REF**: 3mm hole, CustomFootprints:3mm hole, F.Cu at (155.5, 99.5)
- added REF**: 3mm hole, CustomFootprints:3mm hole, F.Cu at (64.0, 160.0)
- added REF**: 3mm hole, CustomFootprints:3mm hole, F.Cu at (227.0, 39.0)
- added REF**: 3mm hole, CustomFootprints:3mm hole, F.Cu at (227.0, 160.0)
- added REF**: 3mm hole, CustomFootprints:3mm hole, F.Cu at (64.0, 39.0)
- added Ref**: Val**, Custom Footprints:seds-logo, F.Cu at (166.2, 87.8)
- R15, R20, R21, R3, R36, R37, R4: value 2.49M -> 2M
- R16, R22, R23, R38, R39, R5, R6: value 487k -> 2M
- R17, R24, R25, R40, R41, R7, R8: value 2M -> 1M
- U2: value MAX33012EASA+ -> 21-0041-3-M_90-0096-8L_MXM
